Commit message: renaming

File: examples/deps/panda_end_effector.urdf (robot description, URDF)
Before this commit: robot panda, 12 links, 11 joints
Links:
- link finger1: geometry collision mesh filename=/home/simon/.julia/dev/Silico.jl/examples/deps/mesh/collisi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; visual mesh filename=/home/simon/.julia/dev/Silico.jl/examples/deps/mesh/visual/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
- link finger2: geometry collision mesh filename=/home/simon/.julia/dev/Silico.jl/examples/deps/mesh/collisi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; visual mesh filename=/home/simon/.julia/dev/Silico.jl/examples/deps/mesh/visual/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
- link link0: geometry collision mesh filename=/home/simon/.julia/dev/Silico.jl/examples/deps/mesh/collisi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; visual mesh filename=/home/simon/.julia/dev/Silico.jl/examples/deps/mesh/visual/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
- link link1: geometry collision mesh filename=/home/simon/.julia/dev/Silico.jl/examples/deps/mesh/collisi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; visual mesh filename=/home/simon/.julia/dev/Silico.jl/examples/deps/mesh/visual/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
- link link2: geometry collision mesh filename=/home/simon/.julia/dev/Silico.jl/examples/deps/mesh/collisi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; visual mesh filename=/home/simon/.julia/dev/Silico.jl/examples/deps/mesh/visual/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
- link link3: geometry collision mesh filename=/home/simon/.julia/dev/Silico.jl/examples/deps/mesh/collisi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; visual mesh filename=/home/simon/.julia/dev/Silico.jl/examples/deps/mesh/visual/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
- link link4: geometry collision mesh filename=/home/simon/.julia/dev/Silico.jl/examples/deps/mesh/collisi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; visual mesh filename=/home/simon/.julia/dev/Silico.jl/examples/deps/mesh/visual/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
- link link5: geometry collision mesh filename=/home/simon/.julia/dev/Silico.jl/examples/deps/mesh/collisi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; visual mesh filename=/home/simon/.julia/dev/Silico.jl/examples/deps/mesh/visual/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
- link link6: geometry collision mesh filename=/home/simon/.julia/dev/Silico.jl/examples/deps/mesh/collisi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; visual mesh filename=/home/simon/.julia/dev/Silico.jl/examples/deps/mesh/visual/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
- link link7: geometry collision mesh filename=/home/simon/.julia/dev/Silico.jl/examples/deps/mesh/collisi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; visual mesh filename=/home/simon/.julia/dev/Silico.jl/examples/deps/mesh/visual/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
- link link8: geometry collision mesh filename=/home/simon/.julia/dev/Silico.jl/examples/deps/mesh/collisi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; visual mesh filename=/home/simon/.julia/dev/Silico.jl/examples/deps/mesh/visual/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
